File: hardware/Kicad_PCB_helios/Microcontroller.sch (KiCad schematic (older format))
At the start: 24 parts, among them U9 ATSAM4S, Y1 16MHz 18pF

Commit message: Dodano 2 zewnętrzne 16 bitowe układy DAC
Podłączono VREF do wewnętrznych DAC

Wszystko działa na jednej magistrali SPI
Connections:
- net !SYNC-X: now reaches U9.29 (PA10/PGMM2)
- net !SYNC-Y: now reaches U9.30 (PA9/PGMM1)
- net !SYNC renamed !SYNC-Quad
- net X renamed X_SCALING
- net Y renamed Y_SCALING
- no-connect marks 36 -> 34
Changed lines of the file:
@@
 EESchema Schematic File Version 2
+LIBS:Helios-rescue
 LIBS:power
 LIBS:device
@@
 Comment4 ""
 $EndDescr
-$Comp
-L ATSAM4S U9
-U 1 1 56B20B8A
-P 7250 2450
-F 0 "U9" H 7250 1137 60  0000 C CNN
-F 1 "ATSAM4S" H 7250 2850 60  0000 C CNN
-F 2 "personal:LQFP-64_10x10mm_Pitch0.5mm" H 7250 2850 60  0001 C CNN
-F 3 "" H 7250 2850 60  0000 C CNN
-	1    7250 2450
-	1    0    0    -1
-$EndComp
 Text HLabel 1850 1300 0    60   UnSpc ~ 0
 3.3V
@@
 $EndComp
 $Comp
-L GND #PWR31
+L GND #PWR039
 U 1 1 56B2611E
 P 2400 2100
-F 0 "#PWR31" H 2400 1850 50  0001 C CNN
+F 0 "#PWR039" H 2400 1850 50  0001 C CNN
 F 1 "GND" H 2400 1950 50  0000 C CNN
 F 2 "" H 2400 2100 50  0000 C CNN
@@
 $EndComp
 $Comp
-L GND #PWR32
+L GND #PWR040
 U 1 1 56B261DD
 P 2500 3400
-F 0 "#PWR32" H 2500 3150 50  0001 C CNN
+F 0 "#PWR040" H 2500 3150 50  0001 C CNN
 F 1 "GND" H 2500 3250 50  0000 C CNN
 F 2 "" H 2500 3400 50  0000 C CNN
@@
 $EndComp
 $Comp
-L GND #PWR33
+L GND #PWR041
 U 1 1 56B264E0
 P 3300 5150
-F 0 "#PWR33" H 3300 4900 50  0001 C CNN
+F 0 "#PWR041" H 3300 4900 50  0001 C CNN
 F 1 "GND" H 3300 5000 50  0000 C CNN
 F 2 "" H 3300 5150 50  0000 C CNN
@@
 $EndComp
 $Comp
-L GND #PWR34
+L GND #PWR042
 U 1 1 56B28207
 P 3600 7400
-F 0 "#PWR34" H 3600 7150 50  0001 C CNN
+F 0 "#PWR042" H 3600 7150 50  0001 C CNN
 F 1 "GND" H 3600 7250 50  0000 C CNN
 F 2 "" H 3600 7400 50  0000 C CNN
@@
 $EndComp
 $Comp
-L GND #PWR35
+L GND #PWR043
 U 1 1 56B282D6
 P 4400 7400
-F 0 "#PWR35" H 4400 7150 50  0001 C CNN
+F 0 "#PWR043" H 4400 7150 50  0001 C CNN
 F 1 "GND" H 4400 7250 50  0000 C CNN
 F 2 "" H 4400 7400 50  0000 C CNN
@@
 SCLK
 Text HLabel 6250 4500 0    60   Output ~ 0
-!SYNC
+!SYNC-Quad
 Text HLabel 8400 4100 2    60   BiDi ~ 0
 D-
@@
 $EndComp
 $Comp
-L GND #PWR36
+L GND #PWR044
 U 1 1 56BC9489
 P 5200 7450
-F 0 "#PWR36" H 5200 7200 50  0001 C CNN
+F 0 "#PWR044" H 5200 7200 50  0001 C CNN
 F 1 "GND" H 5200 7300 50  0000 C CNN
 F 2 "" H 5200 7450 50  0000 C CNN
@@
 $EndComp
 $Comp
-L GND #PWR37
+L GND #PWR045
 U 1 1 56BC94D0
 P 5550 7450
-F 0 "#PWR37" H 5550 7200 50  0001 C CNN
+F 0 "#PWR045" H 5550 7200 50  0001 C CNN
 F 1 "GND" H 5550 7300 50  0000 C CNN
 F 2 "" H 5550 7450 50  0000 C CNN
@@
 VDDIO
 $Comp
-L GND #PWR39
+L GND #PWR046
 U 1 1 56F0F05F
 P 6150 3400
-F 0 "#PWR39" H 6150 3150 50  0001 C CNN
+F 0 "#PWR046" H 6150 3150 50  0001 C CNN
 F 1 "GND" H 6150 3250 50  0000 C CNN
 F 2 "" H 6150 3400 50  0000 C CNN
@@
 VDDIO
 $Comp
-L GND #PWR43
+L GND #PWR047
 U 1 1 56F110A4
 P 8400 4500
-F 0 "#PWR43" H 8400 4250 50  0001 C CNN
+F 0 "#PWR047" H 8400 4250 50  0001 C CNN
 F 1 "GND" H 8400 4350 50  0000 C CNN
 F 2 "" H 8400 4500 50  0000 C CNN
@@
 NRST
 $Comp
-L GND #PWR42
+L GND #PWR048
 U 1 1 56F12B31
 P 8400 3100
-F 0 "#PWR42" H 8400 2850 50  0001 C CNN
+F 0 "#PWR048" H 8400 2850 50  0001 C CNN
 F 1 "GND" H 8400 2950 50  0000 C CNN
 F 2 "" H 8400 3100 50  0000 C CNN
@@
 VDDIN
 $Comp
-L GND #PWR40
+L GND #PWR049
 U 1 1 56F13C65
 P 6200 1900
-F 0 "#PWR40" H 6200 1650 50  0001 C CNN
+F 0 "#PWR049" H 6200 1650 50  0001 C CNN
 F 1 "GND" H 6200 1750 50  0000 C CNN
 F 2 "" H 6200 1900 50  0000 C CNN
@@
 Text Label 3600 6450 0    39   ~ 0
 XIN
-Text HLabel 8400 4400 2    39   Output ~ 0
-X
-Text HLabel 8400 4800 2    39   Output ~ 0
-Y
 Text HLabel 5600 1800 0    60   UnSpc ~ 0
 2.5V
@@
 NoConn ~ 6300 3700
 NoConn ~ 6300 4400
-NoConn ~ 6300 4600
-NoConn ~ 6300 4700
 NoConn ~ 6300 4800
 NoConn ~ 6300 4900
@@
 $EndComp
 $Comp
-L GND #PWR41
+L GND #PWR050
 U 1 1 575A0181
 P 8300 2500
-F 0 "#PWR41" H 8300 2250 50  0001 C CNN
+F 0 "#PWR050" H 8300 2250 50  0001 C CNN
 F 1 "GND" H 8300 2350 50  0000 C CNN
 F 2 "" H 8300 2500 50  0000 C CNN
@@
 NoConn ~ 8400 2400
 $Comp
-L GND #PWR38
+L GND #PWR051
 U 1 1 575C07BB
 P 5750 2200
-F 0 "#PWR38" H 5750 1950 50  0001 C CNN
+F 0 "#PWR051" H 5750 1950 50  0001 C CNN
 F 1 "GND" H 5750 2050 50  0000 C CNN
 F 2 "" H 5750 2200 50  0000 C CNN
@@
 Wire Wire Line
 	5600 1800 6300 1800
-Wire Wire Line
-	8400 4800 8300 4800
 Wire Wire Line
 	8300 4400 8400 4400
@@
 	0    -1   1    0
 $EndComp
+Text HLabel 6300 4600 0    60   Output ~ 0
+!SYNC-X
+Text HLabel 6300 4700 0    60   Output ~ 0
+!SYNC-Y
+$Comp
+L ATSAM4S U9
+U 1 1 56B20B8A
+P 7250 2450
+F 0 "U9" H 7250 1137 60  0000 C CNN
+F 1 "ATSAM4S" H 7250 2850 60  0000 C CNN
+F 2 "personal:LQFP-64_10x10mm_Pitch0.5mm" H 7250 2850 60  0001 C CNN
+F 3 "" H 7250 2850 60  0000 C CNN
+	1    7250 2450
+	1    0    0    -1
+$EndComp
+Wire Wire Line
+	8300 4800 8400 4800
+Text HLabel 8400 4400 2    60   Input ~ 0
+X_SCALING
+Text HLabel 8400 4800 2    60   Input ~ 0
+Y_SCALING
 $EndSCHEMATC

Commit message: Updated PCB Layout
Changed connector to IDC
Parts:
- C19, C20, C21, C22, C25, C26, C27, C28, C32: footprint Capacitors_SMD:C_0402 -> Capacitors_SMD:C_0603
- C29, C31: footprint Capacitors_SMD:C_0402 -> Capacitors_SMD:C_0603_HandSoldering
- ERASE1: footprint Connect:PINHEAD1-2 -> Pin_Headers:Pin_Header_Straight_1x02_Pitch2.54mm
Changed lines of the file:
@@
 F 0 "C21" H 2425 1700 50  0000 L CNN
 F 1 "100nF" H 2425 1500 50  0000 L CNN
-F 2 "Capacitors_SMD:C_0402" H 2438 1450 50  0001 C CNN
+F 2 "Capacitors_SMD:C_0603" H 2438 1450 50  0001 C CNN
 F 3 "" H 2400 1600 50  0000 C CNN
 	1    2400 1600
@@
 $EndComp
 $Comp
-L GND #PWR039
+L GND #PWR044
 U 1 1 56B2611E
 P 2400 2100
-F 0 "#PWR039" H 2400 1850 50  0001 C CNN
+F 0 "#PWR044" H 2400 1850 50  0001 C CNN
 F 1 "GND" H 2400 1950 50  0000 C CNN
 F 2 "" H 2400 2100 50  0000 C CNN
@@
 $EndComp
 $Comp
-L GND #PWR040
+L GND #PWR045
 U 1 1 56B261DD
 P 2500 3400
-F 0 "#PWR040" H 2500 3150 50  0001 C CNN
+F 0 "#PWR045" H 2500 3150 50  0001 C CNN
 F 1 "GND" H 2500 3250 50  0000 C CNN
 F 2 "" H 2500 3400 50  0000 C CNN
@@
 $EndComp
 $Comp
-L GND #PWR041
+L GND #PWR046
 U 1 1 56B264E0
 P 3300 5150
-F 0 "#PWR041" H 3300 4900 50  0001 C CNN
+F 0 "#PWR046" H 3300 4900 50  0001 C CNN
 F 1 "GND" H 3300 5000 50  0000 C CNN
 F 2 "" H 3300 5150 50  0000 C CNN
@@
 F 0 "C29" H 3625 7150 50  0000 L CNN
 F 1 "13pF" H 3625 6950 50  0000 L CNN
-F 2 "Capacitors_SMD:C_0402" H 3638 6900 50  0001 C CNN
+F 2 "Capacitors_SMD:C_0603_HandSoldering" H 3638 6900 50  0001 C CNN
 F 3 "" H 3600 7050 50  0000 C CNN
 	1    3600 7050
@@
 F 0 "C31" H 4425 7150 50  0000 L CNN
 F 1 "13pF" H 4425 6950 50  0000 L CNN
-F 2 "Capacitors_SMD:C_0402" H 4438 6900 50  0001 C CNN
+F 2 "Capacitors_SMD:C_0603_HandSoldering" H 4438 6900 50  0001 C CNN
 F 3 "" H 4400 7050 50  0000 C CNN
 	1    4400 7050
@@
 $EndComp
 $Comp
-L GND #PWR042
+L GND #PWR047
 U 1 1 56B28207
 P 3600 7400
-F 0 "#PWR042" H 3600 7150 50  0001 C CNN
+F 0 "#PWR047" H 3600 7150 50  0001 C CNN
 F 1 "GND" H 3600 7250 50  0000 C CNN
 F 2 "" H 3600 7400 50  0000 C CNN
@@
 $EndComp
 $Comp
-L GND #PWR043
+L GND #PWR048
 U 1 1 56B282D6
 P 4400 7400
-F 0 "#PWR043" H 4400 7150 50  0001 C CNN
+F 0 "#PWR048" H 4400 7150 50  0001 C CNN
 F 1 "GND" H 4400 7250 50  0000 C CNN
 F 2 "" H 4400 7400 50  0000 C CNN
@@
 $EndComp
 $Comp
-L GND #PWR044
+L GND #PWR049
 U 1 1 56BC9489
 P 5200 7450
-F 0 "#PWR044" H 5200 7200 50  0001 C CNN
+F 0 "#PWR049" H 5200 7200 50  0001 C CNN
 F 1 "GND" H 5200 7300 50  0000 C CNN
 F 2 "" H 5200 7450 50  0000 C CNN
@@
 $EndComp
 $Comp
-L GND #PWR045
+L GND #PWR050
 U 1 1 56BC94D0
 P 5550 7450
-F 0 "#PWR045" H 5550 7200 50  0001 C CNN
+F 0 "#PWR050" H 5550 7200 50  0001 C CNN
 F 1 "GND" H 5550 7300 50  0000 C CNN
 F 2 "" H 5550 7450 50  0000 C CNN
@@
 VDDIO
 $Comp
-L GND #PWR046
+L GND #PWR051
 U 1 1 56F0F05F
 P 6150 3400
-F 0 "#PWR046" H 6150 3150 50  0001 C CNN
+F 0 "#PWR051" H 6150 3150 50  0001 C CNN
 F 1 "GND" H 6150 3250 50  0000 C CNN
 F 2 "" H 6150 3400 50  0000 C CNN
@@
 VDDIO
 $Comp
-L GND #PWR047
+L GND #PWR052
 U 1 1 56F110A4
 P 8400 4500
-F 0 "#PWR047" H 8400 4250 50  0001 C CNN
+F 0 "#PWR052" H 8400 4250 50  0001 C CNN
 F 1 "GND" H 8400 4350 50  0000 C CNN
 F 2 "" H 8400 4500 50  0000 C CNN
@@
 NRST
 $Comp
-L GND #PWR048
+L GND #PWR053
 U 1 1 56F12B31
 P 8400 3100
-F 0 "#PWR048" H 8400 2850 50  0001 C CNN
+F 0 "#PWR053" H 8400 2850 50  0001 C CNN
 F 1 "GND" H 8400 2950 50  0000 C CNN
 F 2 "" H 8400 3100 50  0000 C CNN
@@
 VDDIN
 $Comp
-L GND #PWR049
+L GND #PWR054
 U 1 1 56F13C65
 P 6200 1900
-F 0 "#PWR049" H 6200 1650 50  0001 C CNN
+F 0 "#PWR054" H 6200 1650 50  0001 C CNN
 F 1 "GND" H 6200 1750 50  0000 C CNN
 F 2 "" H 6200 1900 50  0000 C CNN
@@
 F 0 "C25" H 2825 1700 50  0000 L CNN
 F 1 "100nF" H 2825 1500 50  0000 L CNN
-F 2 "Capacitors_SMD:C_0402" H 2838 1450 50  0001 C CNN
+F 2 "Capacitors_SMD:C_0603" H 2838 1450 50  0001 C CNN
 F 3 "" H 2800 1600 50  0000 C CNN
 	1    2800 1600
@@
 F 0 "C27" H 3175 1700 50  0000 L CNN
 F 1 "100nF" H 3175 1500 50  0000 L CNN
-F 2 "Capacitors_SMD:C_0402" H 3188 1450 50  0001 C CNN
+F 2 "Capacitors_SMD:C_0603" H 3188 1450 50  0001 C CNN
 F 3 "" H 3150 1600 50  0000 C CNN
 	1    3150 1600
@@
 F 0 "C26" H 2925 3250 50  0000 L CNN
 F 1 "100nF" H 2925 3050 50  0000 L CNN
-F 2 "Capacitors_SMD:C_0402" H 2938 3000 50  0001 C CNN
+F 2 "Capacitors_SMD:C_0603" H 2938 3000 50  0001 C CNN
 F 3 "" H 2900 3150 50  0000 C CNN
 	1    2900 3150
@@
 F 0 "C28" H 3325 4700 50  0000 L CNN
 F 1 "100nF" H 3325 4500 50  0000 L CNN
-F 2 "Capacitors_SMD:C_0402" H 3338 4450 50  0001 C CNN
+F 2 "Capacitors_SMD:C_0603" H 3338 4450 50  0001 C CNN
 F 3 "" H 3300 4600 50  0000 C CNN
 	1    3300 4600
@@
 F 0 "C22" H 2425 4700 50  0000 L CNN
 F 1 "100nF" H 2425 4500 50  0000 L CNN
-F 2 "Capacitors_SMD:C_0402" H 2438 4450 50  0001 C CNN
+F 2 "Capacitors_SMD:C_0603" H 2438 4450 50  0001 C CNN
 F 3 "" H 2400 4600 50  0000 C CNN
 	1    2400 4600
@@
 F 0 "C20" H 2125 4700 50  0000 L CNN
 F 1 "100nF" H 2125 4500 50  0000 L CNN
-F 2 "Capacitors_SMD:C_0402" H 2138 4450 50  0001 C CNN
+F 2 "Capacitors_SMD:C_0603" H 2138 4450 50  0001 C CNN
 F 3 "" H 2100 4600 50  0000 C CNN
 	1    2100 4600
@@
 F 0 "C19" H 1825 4700 50  0000 L CNN
 F 1 "100nF" H 1825 4500 50  0000 L CNN
-F 2 "Capacitors_SMD:C_0402" H 1838 4450 50  0001 C CNN
+F 2 "Capacitors_SMD:C_0603" H 1838 4450 50  0001 C CNN
 F 3 "" H 1800 4600 50  0000 C CNN
 	1    1800 4600
@@
 $EndComp
 $Comp
-L GND #PWR050
+L GND #PWR055
 U 1 1 575A0181
 P 8300 2500
-F 0 "#PWR050" H 8300 2250 50  0001 C CNN
+F 0 "#PWR055" H 8300 2250 50  0001 C CNN
 F 1 "GND" H 8300 2350 50  0000 C CNN
 F 2 "" H 8300 2500 50  0000 C CNN
@@
 NoConn ~ 8400 2400
 $Comp
-L GND #PWR051
+L GND #PWR056
 U 1 1 575C07BB
 P 5750 2200
-F 0 "#PWR051" H 5750 1950 50  0001 C CNN
+F 0 "#PWR056" H 5750 1950 50  0001 C CNN
 F 1 "GND" H 5750 2050 50  0000 C CNN
 F 2 "" H 5750 2200 50  0000 C CNN
@@
 F 0 "C32" H 5775 2150 50  0000 L CNN
 F 1 "13pF" H 5775 1950 50  0000 L CNN
-F 2 "Capacitors_SMD:C_0402" H 5788 1900 50  0001 C CNN
+F 2 "Capacitors_SMD:C_0603" H 5788 1900 50  0001 C CNN
 F 3 "" H 5750 2050 50  0000 C CNN
 	1    5750 2050
@@
 Wire Wire Line
 	3300 4400 3900 4400
-$Comp
-L CONN_01X02 ERASE1
-U 1 1 5792C984
-P 1150 7250
-F 0 "ERASE1" H 1150 7400 50  0000 C CNN
-F 1 "CONN_01X02" V 1250 7250 50  0000 C CNN
-F 2 "Connect:PINHEAD1-2" H 1150 7250 50  0001 C CNN
-F 3 "" H 1150 7250 50  0000 C CNN
-	1    1150 7250
-	0    -1   1    0
-$EndComp
 Text HLabel 6300 4600 0    60   Output ~ 0
 !SYNC-X
@@
 Text HLabel 8400 4800 2    60   Input ~ 0
 Y_SCALING
+$Comp
+L CONN_01X02 ERASE1
+U 1 1 5792C984
+P 1150 7250
+F 0 "ERASE1" H 1150 7400 50  0000 C CNN
+F 1 "CONN_01X02" V 1250 7250 50  0000 C CNN
+F 2 "Pin_Headers:Pin_Header_Straight_1x02_Pitch2.54mm" H 1150 7250 50  0001 C CNN
+F 3 "" H 1150 7250 50  0000 C CNN
+	1    1150 7250
+	0    -1   1    0
+$EndComp
 $EndSCHEMATC
